Commit message: started gazebo

File: description/robot.urdf.xacro (robot description, xacro)
@@ -3,3 +3,4 @@
     <xacro:include filename="material.xacro"/>
     <xacro:include filename="robot_core.xacro"/>
+    <xacro:include filename="gazebo_control.xacro" />
 </robot>

File: description/robot_core.xacro (robot description, xacro)
@@ -4,4 +4,7 @@
     <!-- base link -->
     <link name="base_link">
+        <!-- <xacro:inertial_sphere mass="0.01" radius="0.01">
+            <origin xyz="0 0 0" rpy="0 0 0"/>
+        </xacro:inertial_sphere> -->
     </link>
     <!-- chassis link -->
@@ -9,5 +12,5 @@
         <parent link="base_link"/>
         <child link="chassis"/>
-        <origin xyz="-0.1 0.0 0.0"/>
+        <origin xyz="-0.1 0.0 0"/>
     </joint>
     <link name="chassis">
@@ -29,4 +32,7 @@
         </xacro:inertial_box>
     </link>
+    <gazebo reference = "chassis">
+        <material>Gazebo/White</material>
+    </gazebo>
     <!-- left wheel link -->
      <joint name="left_wheel_joint" type="continuous">
@@ -52,6 +58,9 @@
         </xacro:inertial_cylinder>
      </link>
+     <gazebo reference = "left_wheel">
+        <material>Gazebo/Black</material>
+    </gazebo>
     <!-- right wheel link -->
-     <joint name="right_wheel_link" type="continuous">
+     <joint name="right_wheel_joint" type="continuous">
         <parent link="base_link"/>
         <child link="right_wheel"/>
@@ -75,4 +84,7 @@
         </xacro:inertial_cylinder>
      </link>
+     <gazebo reference = "right_wheel">
+        <material>Gazebo/Black</material>
+    </gazebo>
     <!-- caster wheel link-->
      <joint name="caster_wheel_link" type="fixed">
@@ -97,3 +109,8 @@
         </xacro:inertial_sphere>
      </link>
+     <gazebo reference = "caster_wheel">
+        <material>Gazebo/Yellow</material>
+        <mu1 value = "0.001"/>
+        <mu2 value = "0.001"/>
+    </gazebo>
 </robot>
