Commit message: added lidar

File: description/material.xacro (robot description, xacro)
@@ -13,3 +13,6 @@
         <color rgba="0.75 0.75 0.75 1.0"/>
    </material>
+   <material name="red">
+        <color rgba="1 0.0 0.0 1.0"/>
+   </material>
 </robot>

File: description/robot.urdf.xacro (robot description, xacro)
@@ -4,3 +4,4 @@
     <xacro:include filename="robot_core.xacro"/>
     <xacro:include filename="gazebo_control.xacro" />
+    <xacro:include filename="lidar.xacro" />
 </robot>
