Commit message: added controller manager

File: description/camera.xacro (robot description, xacro)
@@ -15,5 +15,5 @@
         <collision>
             <geometry>
-                <box size="0.01, 0.03 0.03"/>
+                <box size="0.01 0.03 0.03"/>
             </geometry>
         </collision>

File: description/robot.urdf.xacro (robot description, xacro)
@@ -3,6 +3,7 @@
     <xacro:include filename="material.xacro"/>
     <xacro:include filename="robot_core.xacro"/>
-    <xacro:include filename="gazebo_control.xacro" />
+    <!-- <xacro:include filename="gazebo_control.xacro" /> -->
     <xacro:include filename="lidar.xacro" />
     <xacro:include filename="camera.xacro" />
+    <xacro:include filename="ros2_control.xacro" />
 </robot>
