Commit message: changed to arduino control, added header

File: description/ros2_control.xacro (robot description, xacro)
@@ -1,5 +1,5 @@
 <?xml version="1.0"?>
 <robot xmlns:xacro="http://www.ros.org/wiki/xacro"  name="robot">
-    <ros2_control name = "Gazebo_system" type = "system">
+    <!-- <ros2_control name = "Gazebo_system" type = "system">
         <hardware>
             <plugin>gz_ros2_control/GazeboSimSystem</plugin>
@@ -27,4 +27,29 @@
             <controller_manager_prefix_node_name>controller_manager</controller_manager_prefix_node_name>
         </plugin>
-    </gazebo>
+    </gazebo> -->
+    <ros2_control name = "arduino_drive" type = "system">
+        <hardware>
+            <plugin>my_bot/MyBotArduinoHardware</plugin>
+            <param name="device">/dev/ttyACM0</param> <!--change this to the correct USB-->
+            <param name="baud_rate">115200</param>
+            <param name="timeout_ms">1000</param>
+            <param name="enc_counts_per_rev">330</param>
+        </hardware>
+        <joint name="left_wheel_joint">
+            <command_interface name="velocity">
+                <param name="min">-10</param>
+                <param name="max">10</param>
+            </command_interface>
+            <state_interface name = "velocity"/>
+            <state_interface name = "position"/>
+        </joint>
+        <joint name="right_wheel_joint">
+            <command_interface name="velocity">
+                <param name="min">-10</param>
+                <param name="max">10</param>
+            </command_interface>
+            <state_interface name = "velocity"/>
+            <state_interface name = "position"/>
+        </joint>
+    </ros2_control>
 </robot>
