Commit message: ready for pi

File: description/robot_core.xacro (robot description, xacro)
@@ -45,5 +45,5 @@
         <visual>
             <geometry>
-                <cylinder radius="0.05" length="0.04"/>
+                <cylinder radius="0.085" length="0.04"/>
             </geometry>
             <material name="black"/>
@@ -71,5 +71,5 @@
         <visual>
             <geometry>
-                <cylinder radius="0.05" length="0.04"/>
+                <cylinder radius="0.08s" length="0.04"/>
             </geometry>
             <material name="black"/>

File: description/ros2_control_real.xacro (robot description, xacro)
@@ -1,31 +1,4 @@
 <?xml version="1.0"?>
 <robot xmlns:xacro="http://www.ros.org/wiki/xacro"  name="robot">
-    <!-- <ros2_control name = "Gazebo_system" type = "system">
-        <hardware>
-            <plugin>gz_ros2_control/GazeboSimSystem</plugin>
-        </hardware>
-        <joint name="left_wheel_joint">
-            <command_interface name="velocity">
-                <param name="min">-10</param>
-                <param name="max">10</param>
-            </command_interface>
-            <state_interface name = "velocity"/>
-            <state_interface name = "position"/>
-        </joint>
-        <joint name="right_wheel_joint">
-            <command_interface name="velocity">
-                <param name="min">-10</param>
-                <param name="max">10</param>
-            </command_interface>
-            <state_interface name = "velocity"/>
-            <state_interface name = "position"/>
-        </joint>
-    </ros2_control>
-    <gazebo>
-        <plugin filename="libgz_ros2_control-system.so" name="gz_ros2_control::GazeboSimROS2ControlPlugin">
-            <parameters>/home/jrm/dev_ws/src/my_bot/config/my_controllers.yaml</parameters>
-            <controller_manager_prefix_node_name>controller_manager</controller_manager_prefix_node_name>
-        </plugin>
-    </gazebo> -->
     <ros2_control name = "arduino_drive" type = "system">
         <hardware>
@@ -34,5 +7,5 @@
             <param name="baud_rate">115200</param>
             <param name="timeout_ms">1000</param>
-            <param name="enc_counts_per_rev">330</param>
+            <param name="enc_counts_per_rev">615</param>
         </hardware>
         <joint name="left_wheel_joint">

Commit message: fix minor issue

File: description/robot_core.xacro (robot description, xacro)
@@ -71,5 +71,5 @@
         <visual>
             <geometry>
-                <cylinder radius="0.08s" length="0.04"/>
+                <cylinder radius="0.085" length="0.04"/>
             </geometry>
             <material name="black"/>
